File: kimchi-gps-lid.kicad_pcb (KiCad board)
At the start: 4 copper layers, 65 x 32 mm, 22 parts, among them J1 DF40HC(3.5)-60DS, J2 DF40HC(3.5)-60DS, Q1 DTC143ZEBTL, Q2 DTC143ZEBTL, U1 24C32, U2 L80RE-M37, U3 TXS0104ED

Commit message: Added oshpark and group gets logo to silkscreen
Parts:
- added G***: LOGO, logo:oshpark_logo, B.Cu at (151.8, 106.8)
- added G***: LOGO, logo:groupgets_logo, B.Cu at (163.6, 106.8)
Other:
- board text added: "GPS Module"
- board text added: "Level Shifter"
- board text added: "Thanks to OSHpark and GroupGets for making this board possible"

Commit message: Changed value of LED resistor according to requirements of green LED
Parts:
- R2: value R -> 690
